File: SENSORES.kicad_sch (KiCad schematic)
At the start: 47 parts, among them J10 RELES_2, J11 Throttle, J12 I2C_EXT1, J13 I2C_EXT2, J14 S_HALL, J15 RF_PPM, J17 SERVO2, J18 SERVO1, J19 +7V_IN, J2 S_GIRO, J6 IBT_2, J7 FC1, J8 FC2, J9 RELES_1, U4 BMI088, U5 74HC595, U6 ULN2003A, U7 LM358

Commit message: routing
Parts:
- R2, R3: value R -> 4.7k
Changed lines of the file:
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@@
 			)
 		)
-		(property "Value" "R"
+		(property "Value" "4.7k"
 			(at 187.96 35.5599 0)
 			(show_name no)
@@
 			)
 		)
-		(property "Value" "R"
+		(property "Value" "4.7k"
 			(at 187.96 66.0399 0)
 			(show_name no)

Commit message: routeo terminado v1
Changed lines of the file:
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@@
 		(lib_id "Device:C")
 		(at 60.96 130.81 0)
+		(mirror y)
 		(unit 1)
 		(body_style 1)
@@
 		(dnp no)
 		(property "Reference" "C21"
-			(at 63.754 131.572 0)
+			(at 58.166 131.572 0)
 			(show_name no)
 			(do_not_autoplace no)
@@
 		)
 		(property "Value" "100nF"
-			(at 63.754 134.112 0)
+			(at 58.166 134.112 0)
 			(show_name no)
 			(do_not_autoplace no)
@@
 		)
 		(property "Footprint" "Capacitor_SMD:C_0603_1608Metric"
-			(at 61.9252 134.62 0)
+			(at 59.9948 134.62 0)
 			(hide yes)
 			(show_name no)
@@
 		)
 		(property "LCSC PN" "C1590"
-			(at 0 0 0)
+			(at 121.92 0 0)
 			(hide yes)
 			(show_name no)
@@
 		)
 		(property "Manufacturer" "Samsung Electro-Mechanics"
-			(at 0 0 0)
+			(at 121.92 0 0)
 			(hide yes)
 			(show_name no)
@@
 		)
 		(property "MPN" "CL10B104KA8NNNC"
-			(at 0 0 0)
+			(at 121.92 0 0)
 			(hide yes)
 			(show_name no)

Commit message: presupuesto
Parts:
- R2, R3: BOM Comments Valor pendiente: no seleccionar ni montar hasta definir el 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 -> Componente confirmado: resistencia pull-up de 4.7 kOhm, 060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; LCSC PN (none) -> C23162; MPN (none) -> 0603WAF4701T5E; Manufacturer (none) -> Walsin Technology
Changed lines of the file:
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@@
 			)
 		)
-		(property "Datasheet" ""
-			(at 26.67 106.68 0)
+		(property "MPN" "0603WAF4701T5E"
+			(at 0 0 0)
 			(hide yes)
 			(show_name no)
@@
 			)
 		)
-		(property "Description" "Resistor"
-			(at 26.67 106.68 0)
+		(property "Manufacturer" "Walsin Technology"
+			(at 0 0 0)
 			(hide yes)
 			(show_name no)
@@
 			)
 		)
-		(property "Manufacturer" "Walsin Technology"
-			(at 0 0 0)
+		(property "Datasheet" ""
+			(at 26.67 106.68 0)
 			(hide yes)
 			(show_name no)
@@
 			)
 		)
-		(property "MPN" "0603WAF4701T5E"
-			(at 0 0 0)
+		(property "Description" "Resistor"
+			(at 26.67 106.68 0)
 			(hide yes)
 			(show_name no)
@@
 			)
 		)
+		(property "MPN" "0603WAF4701T5E"
+			(at 0 0 0)
+			(hide yes)
+			(show_name no)
+			(do_not_autoplace no)
+			(effects
+				(font
+					(size 1.27 1.27)
+				)
+			)
+		)
+		(property "Manufacturer" "Walsin Technology"
+			(at 0 0 0)
+			(hide yes)
+			(show_name no)
+			(do_not_autoplace no)
+			(effects
+				(font
+					(size 1.27 1.27)
+				)
+			)
+		)
+		(property "LCSC PN" "C23162"
+			(at 0 0 0)
+			(hide yes)
+			(show_name no)
+			(do_not_autoplace no)
+			(effects
+				(font
+					(size 1.27 1.27)
+				)
+			)
+		)
 		(property "Datasheet" ""
 			(at 185.42 34.29 0)
@@
 			)
 		)
-		(property "BOM Comments" "Valor pendiente: no seleccionar ni montar hasta definir el requisito eléctrico."
+		(property "BOM Comments" "Componente confirmado: resistencia pull-up de 4.7 kOhm, 0603, LCSC C23162."
 			(at 0 0 0)
 			(hide yes)
@@
 			)
 		)
+		(property "MPN" "0603WAF4701T5E"
+			(at 0 0 0)
+			(hide yes)
+			(show_name no)
+			(do_not_autoplace no)
+			(effects
+				(font
+					(size 1.27 1.27)
+				)
+			)
+		)
+		(property "Manufacturer" "Walsin Technology"
+			(at 0 0 0)
+			(hide yes)
+			(show_name no)
+			(do_not_autoplace no)
+			(effects
+				(font
+					(size 1.27 1.27)
+				)
+			)
+		)
+		(property "LCSC PN" "C23162"
+			(at 0 0 0)
+			(hide yes)
+			(show_name no)
+			(do_not_autoplace no)
+			(effects
+				(font
+					(size 1.27 1.27)
+				)
+			)
+		)
 		(property "Datasheet" ""
 			(at 185.42 64.77 0)
@@
 			)
 		)
-		(property "BOM Comments" "Valor pendiente: no seleccionar ni montar hasta definir el requisito eléctrico."
+		(property "BOM Comments" "Componente confirmado: resistencia pull-up de 4.7 kOhm, 0603, LCSC C23162."
 			(at 0 0 0)
 			(hide yes)
