File: SENSORES.kicad_sch (KiCad schematic)
At the start: 47 parts, among them J10 RELES_2, J11 Throttle, J12 I2C_EXT1, J13 I2C_EXT2, J14 S_HALL, J15 RF_PPM, J17 SERVO2, J18 SERVO1, J19 +7V_IN, J2 S_GIRO, J6 IBT_2, J7 FC1, J8 FC2, J9 RELES_1, U4 BMI088, U5 74HC595, U6 ULN2003A, U7 LM358

Commit message: fixes
Parts:
- J10, J11, J12, J13, J14, J15, J17, J18, J19, J2, J6, J7, J8, J9: now left out of the parts list
Changed lines of the file:
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@@
 		(body_style 1)
 		(exclude_from_sim no)
-		(in_bom yes)
+		(in_bom no)
 		(on_board yes)
-		(in_pos_files yes)
+		(in_pos_files no)
 		(dnp no)
 		(fields_autoplaced yes)
@@
 		(body_style 1)
 		(exclude_from_sim no)
-		(in_bom yes)
+		(in_bom no)
 		(on_board yes)
-		(in_pos_files yes)
+		(in_pos_files no)
 		(dnp no)
 		(fields_autoplaced yes)
@@
 		(body_style 1)
 		(exclude_from_sim no)
-		(in_bom yes)
+		(in_bom no)
 		(on_board yes)
-		(in_pos_files yes)
+		(in_pos_files no)
 		(dnp no)
 		(fields_autoplaced yes)
@@
 		(body_style 1)
 		(exclude_from_sim no)
-		(in_bom yes)
+		(in_bom no)
 		(on_board yes)
-		(in_pos_files yes)
+		(in_pos_files no)
 		(dnp no)
 		(fields_autoplaced yes)
@@
 		(body_style 1)
 		(exclude_from_sim no)
-		(in_bom yes)
+		(in_bom no)
 		(on_board yes)
-		(in_pos_files yes)
+		(in_pos_files no)
 		(dnp no)
 		(fields_autoplaced yes)
@@
 		(body_style 1)
 		(exclude_from_sim no)
-		(in_bom yes)
+		(in_bom no)
 		(on_board yes)
-		(in_pos_files yes)
+		(in_pos_files no)
 		(dnp no)
 		(property "Reference" "J11"
@@
 		(body_style 1)
 		(exclude_from_sim no)
-		(in_bom yes)
+		(in_bom no)
 		(on_board yes)
-		(in_pos_files yes)
+		(in_pos_files no)
 		(dnp no)
 		(fields_autoplaced yes)
@@
 		(body_style 1)
 		(exclude_from_sim no)
-		(in_bom yes)
+		(in_bom no)
 		(on_board yes)
-		(in_pos_files yes)
+		(in_pos_files no)
 		(dnp no)
 		(fields_autoplaced yes)
@@
 		(body_style 1)
 		(exclude_from_sim no)
-		(in_bom yes)
+		(in_bom no)
 		(on_board yes)
-		(in_pos_files yes)
+		(in_pos_files no)
 		(dnp no)
 		(property "Reference" "J6"
@@
 		(body_style 1)
 		(exclude_from_sim no)
-		(in_bom yes)
+		(in_bom no)
 		(on_board yes)
-		(in_pos_files yes)
+		(in_pos_files no)
 		(dnp no)
 		(property "Reference" "J13"
@@
 		(body_style 1)
 		(exclude_from_sim no)
-		(in_bom yes)
+		(in_bom no)
 		(on_board yes)
-		(in_pos_files yes)
+		(in_pos_files no)
 		(dnp no)
 		(property "Reference" "J12"
@@
 		(body_style 1)
 		(exclude_from_sim no)
-		(in_bom yes)
+		(in_bom no)
 		(on_board yes)
-		(in_pos_files yes)
+		(in_pos_files no)
 		(dnp no)
 		(fields_autoplaced yes)
@@
 		(body_style 1)
 		(exclude_from_sim no)
-		(in_bom yes)
+		(in_bom no)
 		(on_board yes)
-		(in_pos_files yes)
+		(in_pos_files no)
 		(dnp no)
 		(fields_autoplaced yes)
@@
 		(body_style 1)
 		(exclude_from_sim no)
-		(in_bom yes)
+		(in_bom no)
 		(on_board yes)
-		(in_pos_files yes)
+		(in_pos_files no)
 		(dnp no)
 		(fields_autoplaced yes)

Commit message: Consolida pasivos Basic y valida filtro de acelerador
Parts:
- C12, C13, C15: LCSC PN C1590 -> C14663; MPN CL10B104KA8NNNC -> CC0603KRX7R9BB104; Manufacturer Samsung Electro-Mechanics -> Yageo; Manufacturer Part CL10B104KA8NNNC -> CC0603KRX7R9BB104
- C17, C18, C19, C21: LCSC PN C1590 -> C14663; MPN CL10B104KA8NNNC -> CC0603KRX7R9BB104; Manufacturer Samsung Electro-Mechanics -> Yageo; Manufacturer Part (none) -> CC0603KRX7R9BB104
- C20: value 1uF -> 100nF; LCSC PN C108463 -> C14663; MPN 0603B105K160CT -> CC0603KRX7R9BB104; Manufacturer Walsin Technology -> Yageo; Manufacturer Part (none) -> CC0603KRX7R9BB104
- R17: value 4.7k -> 47k; LCSC PN C23162 -> C25819; MPN 0603WAF4701T5E -> 0603WAF4702T5E; Manufacturer Walsin Technology -> UNI-ROYAL; Manufacturer Part (none) -> 0603WAF4702T5E
Changed lines of the file:
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@@
 			)
 		)
-		(property "Value" "4.7k"
+		(property "Value" "47k"
 			(at 26.67 102.87 90)
 			(show_name no)
@@
 			)
 		)
-		(property "MPN" "0603WAF4701T5E"
+		(property "MPN" "0603WAF4702T5E"
 			(at 0 0 0)
 			(hide yes)
@@
 			)
 		)
-		(property "Manufacturer" "Walsin Technology"
+		(property "Manufacturer" "UNI-ROYAL"
 			(at 0 0 0)
 			(hide yes)
@@
 			)
 		)
-		(property "LCSC PN" "C23162"
+		(property "LCSC PN" "C25819"
 			(at 0 0 0)
 			(hide yes)
@@
 			)
 		)
+		(property "Manufacturer Part" "0603WAF4702T5E" (at 0 0 0)
+			(effects
+				(font
+					(size 1.27 1.27)
+				)
+				(hide yes)
+			)
+		)
 		(pin "1"
 		)
@@
 			)
 		)
-		(property "LCSC PN" "C1590"
+		(property "LCSC PN" "C14663"
 			(at 0 0 0)
 			(hide yes)
@@
 			)
 		)
-		(property "Manufacturer" "Samsung Electro-Mechanics"
+		(property "Manufacturer" "Yageo"
 			(at 0 0 0)
 			(hide yes)
@@
 			)
 		)
-		(property "Manufacturer Part" "CL10B104KA8NNNC"
+		(property "Manufacturer Part" "CC0603KRX7R9BB104"
 			(at 0 0 0)
 			(hide yes)
@@
 			)
 		)
-		(property "MPN" "CL10B104KA8NNNC"
+		(property "MPN" "CC0603KRX7R9BB104"
 			(at 0 0 0)
 			(hide yes)
@@
 			)
 		)
-		(property "LCSC PN" "C1590"
+		(property "LCSC PN" "C14663"
 			(at 0 0 0)
 			(hide yes)
@@
 			)
 		)
-		(property "Manufacturer" "Samsung Electro-Mechanics"
+		(property "Manufacturer" "Yageo"
 			(at 0 0 0)
 			(hide yes)
@@
 			)
 		)
-		(property "Manufacturer Part" "CL10B104KA8NNNC"
+		(property "Manufacturer Part" "CC0603KRX7R9BB104"
 			(at 0 0 0)
 			(hide yes)
@@
 			)
 		)
-		(property "MPN" "CL10B104KA8NNNC"
+		(property "MPN" "CC0603KRX7R9BB104"
 			(at 0 0 0)
 			(hide yes)
@@
 			)
 		)
-		(property "LCSC PN" "C1590"
+		(property "LCSC PN" "C14663"
 			(at 0 0 0)
 			(hide yes)
@@
 			)
 		)
-		(property "Manufacturer" "Samsung Electro-Mechanics"
+		(property "Manufacturer" "Yageo"
 			(at 0 0 0)
 			(hide yes)
@@
 			)
 		)
-		(property "MPN" "CL10B104KA8NNNC"
+		(property "MPN" "CC0603KRX7R9BB104"
 			(at 0 0 0)
 			(hide yes)
@@
 			)
 		)
+		(property "Manufacturer Part" "CC0603KRX7R9BB104" (at 0 0 0)
+			(effects
+				(font
+					(size 1.27 1.27)
+				)
+				(hide yes)
+			)
+		)
 		(pin "1"
 		)
@@
 			)
 		)
-		(property "LCSC PN" "C1590"
+		(property "LCSC PN" "C14663"
 			(at 0 0 0)
 			(hide yes)
@@
 			)
 		)
-		(property "Manufacturer" "Samsung Electro-Mechanics"
+		(property "Manufacturer" "Yageo"
 			(at 0 0 0)
 			(hide yes)
@@
 			)
 		)
-		(property "MPN" "CL10B104KA8NNNC"
+		(property "MPN" "CC0603KRX7R9BB104"
 			(at 0 0 0)
 			(hide yes)
@@
 			)
 		)
+		(property "Manufacturer Part" "CC0603KRX7R9BB104" (at 0 0 0)
+			(effects
+				(font
+					(size 1.27 1.27)
+				)
+				(hide yes)
+			)
+		)
 		(pin "1"
 		)
@@
 			)
 		)
-		(property "LCSC PN" "C1590"
+		(property "LCSC PN" "C14663"
 			(at 121.92 0 0)
 			(hide yes)
@@
 			)
 		)
-		(property "Manufacturer" "Samsung Electro-Mechanics"
+		(property "Manufacturer" "Yageo"
 			(at 121.92 0 0)
 			(hide yes)
@@
 			)
 		)
-		(property "MPN" "CL10B104KA8NNNC"
+		(property "MPN" "CC0603KRX7R9BB104"
 			(at 121.92 0 0)
 			(hide yes)
@@
 			)
 		)
+		(property "Manufacturer Part" "CC0603KRX7R9BB104" (at 0 0 0)
+			(effects
+				(font
+					(size 1.27 1.27)
+				)
+				(hide yes)
+			)
+		)
 		(pin "1"
 		)
@@
 			)
 		)
-		(property "LCSC PN" "C1590"
+		(property "LCSC PN" "C14663"
 			(at 196.85 76.2 0)
 			(hide yes)
@@
 			)
 		)
-		(property "Manufacturer" "Samsung Electro-Mechanics"
+		(property "Manufacturer" "Yageo"
 			(at 196.85 76.2 0)
 			(hide yes)
@@
 			)
 		)
-		(property "Manufacturer Part" "CL10B104KA8NNNC"
+		(property "Manufacturer Part" "CC0603KRX7R9BB104"
 			(at 196.85 76.2 0)
 			(hide yes)
@@
 			)
 		)
-		(property "MPN" "CL10B104KA8NNNC"
+		(property "MPN" "CC0603KRX7R9BB104"
 			(at 196.85 76.2 0)
 			(hide yes)
@@
 			)
 		)
-		(property "Value" "1uF"
+		(property "Value" "100nF"
 			(at 34.29 121.9199 0)
 			(show_name no)
@@
 			)
 		)
-		(property "LCSC PN" "C108463"
+		(property "LCSC PN" "C14663"
 			(at 0 0 0)
 			(hide yes)
@@
 			)
 		)
-		(property "Manufacturer" "Walsin Technology"
+		(property "Manufacturer" "Yageo"
 			(at 0 0 0)
 			(hide yes)
@@
 			)
 		)
-		(property "MPN" "0603B105K160CT"
+		(property "MPN" "CC0603KRX7R9BB104"
 			(at 0 0 0)
 			(hide yes)
@@
 			)
 		)
+		(property "Manufacturer Part" "CC0603KRX7R9BB104" (at 0 0 0)
+			(effects
+				(font
+					(size 1.27 1.27)
+				)
+				(hide yes)
+			)
+		)
 		(pin "1"
 		)
@@
 			)
 		)
-		(property "LCSC PN" "C1590"
+		(property "LCSC PN" "C14663"
 			(at 0 0 0)
 			(hide yes)
@@
 			)
 		)
-		(property "Manufacturer" "Samsung Electro-Mechanics"
+		(property "Manufacturer" "Yageo"
 			(at 0 0 0)
 			(hide yes)
@@
 			)
 		)
-		(property "MPN" "CL10B104KA8NNNC"
+		(property "MPN" "CC0603KRX7R9BB104"
 			(at 0 0 0)
 			(hide yes)
@@
 			)
 		)
+		(property "Manufacturer Part" "CC0603KRX7R9BB104" (at 0 0 0)
+			(effects
+				(font
+					(size 1.27 1.27)
+				)
+				(hide yes)
+			)
+		)

Commit message: Actualiza C14 y C16 con alternativa Basic disponible y registra cotizacion
Parts:
- C14, C16: LCSC PN C107125 -> C1779; MPN CC0805KKX5R6BB475 -> CL21A475KAQNNNE; Manufacturer YAGEO -> Samsung Electro-Mechanics; Manufacturer Part CC0805KKX5R6BB475 -> CL21A475KAQNNNE
Changed lines of the file:
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@@
 			)
 		)
-		(property "Datasheet" ""
+		(property "Datasheet" "https://media.digikey.com/pdf/Data%20Sheets/Samsung%20PDFs/CL21A475KAQNNNE_Spec.pdf"
 			(at 128.27 34.29 0)
 			(hide yes)
@@
 			)
 		)
-		(property "LCSC PN" "C107125"
+		(property "LCSC PN" "C1779"
 			(at 71.12 -1.27 0)
 			(hide yes)
@@
 			)
 		)
-		(property "Manufacturer" "YAGEO"
+		(property "Manufacturer" "Samsung Electro-Mechanics"
 			(at 71.12 -1.27 0)
 			(hide yes)
@@
 			)
 		)
-		(property "Manufacturer Part" "CC0805KKX5R6BB475"
+		(property "Manufacturer Part" "CL21A475KAQNNNE"
 			(at 71.12 -1.27 0)
 			(hide yes)
@@
 			)
 		)
-		(property "MPN" "CC0805KKX5R6BB475"
+		(property "MPN" "CL21A475KAQNNNE"
 			(at 71.12 -1.27 0)
 			(hide yes)
@@
 			)
 		)
-		(property "Datasheet" ""
+		(property "Datasheet" "https://media.digikey.com/pdf/Data%20Sheets/Samsung%20PDFs/CL21A475KAQNNNE_Spec.pdf"
 			(at 57.15 35.56 0)
 			(hide yes)
@@
 			)
 		)
-		(property "LCSC PN" "C107125"
+		(property "LCSC PN" "C1779"
 			(at 0 0 0)
 			(hide yes)
@@
 			)
 		)
-		(property "Manufacturer" "YAGEO"
+		(property "Manufacturer" "Samsung Electro-Mechanics"
 			(at 0 0 0)
 			(hide yes)
@@
 			)
 		)
-		(property "Manufacturer Part" "CC0805KKX5R6BB475"
+		(property "Manufacturer Part" "CL21A475KAQNNNE"
 			(at 0 0 0)
 			(hide yes)
@@
 			)
 		)
-		(property "MPN" "CC0805KKX5R6BB475"
+		(property "MPN" "CL21A475KAQNNNE"
 			(at 0 0 0)
 			(hide yes)
