File: PCB_SALUS_v3.kicad_pcb (KiCad board)
At the start: 2 copper layers, 100 x 100 mm, 87 parts, among them J1 Debug_U0, J10 RELES_2, J11 Throttle, J12 I2C_EXT1, J13 I2C_EXT2, J14 S_HALL, J15 RF_PPM, J16 USB_NATIVO, J17 SERVO2, J18 SERVO1, J19 +7V_IN, J2 S_GIRO, J20 3V_IN, J21 RS485, J22 GPIOS_AUX, J3 RS485, J4 Uart1, J5 5V_IN, J6 IBT_2, J7 FC1, J8 FC2, J9 RELES_1, U1 AMS1117CD-3.3, U2 SP3485EN, U4 BMI088, U5 74HC595, U6 ULN2003A, U7 LM358, U8 ESP32-S3-WROOM-1

Commit message: Consolida pasivos Basic y valida filtro de acelerador
Parts:
- C20: value 1uF -> 100nF
- R17: value 4.7k -> 47k
Changed lines of the file:
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@@
 			)
 		)
-		(property "LCSC PN" "C1590"
+		(property "LCSC PN" "C14663"
 			(at 0 0 90)
 			(unlocked yes)
@@
 			)
 		)
-		(property "Manufacturer" "Samsung Electro-Mechanics"
+		(property "Manufacturer" "Yageo"
 			(at 0 0 90)
 			(unlocked yes)
@@
 			)
 		)
-		(property "Manufacturer Part" "CL10B104KA8NNNC"
+		(property "Manufacturer Part" "CC0603KRX7R9BB104"
 			(at 0 0 90)
 			(unlocked yes)
@@
 			)
 		)
-		(property "MPN" "CL10B104KA8NNNC"
+		(property "MPN" "CC0603KRX7R9BB104"
 			(at 0 0 90)
 			(unlocked yes)
@@
 			)
 		)
-		(property "LCSC PN" "C1590"
+		(property "LCSC PN" "C14663"
 			(at 0 0 90)
 			(unlocked yes)
@@
 			)
 		)
-		(property "Manufacturer" "Samsung Electro-Mechanics"
+		(property "Manufacturer" "Yageo"
 			(at 0 0 90)
 			(unlocked yes)
@@
 			)
 		)
-		(property "Manufacturer Part" "CL10B104KA8NNNC"
+		(property "Manufacturer Part" "CC0603KRX7R9BB104"
 			(at 0 0 90)
 			(unlocked yes)
@@
 			)
 		)
-		(property "MPN" "CL10B104KA8NNNC"
+		(property "MPN" "CC0603KRX7R9BB104"
 			(at 0 0 90)
 			(unlocked yes)
@@
 			)
 		)
-		(property "LCSC PN" "C1590"
+		(property "LCSC PN" "C14663"
 			(at 0 0 270)
 			(unlocked yes)
@@
 			)
 		)
-		(property "Manufacturer" "Samsung Electro-Mechanics"
+		(property "Manufacturer" "Yageo"
 			(at 0 0 270)
 			(unlocked yes)
@@
 			)
 		)
-		(property "Manufacturer Part" "CL10B104KA8NNNC"
+		(property "Manufacturer Part" "CC0603KRX7R9BB104"
 			(at 0 0 270)
 			(unlocked yes)
@@
 			)
 		)
-		(property "MPN" "CL10B104KA8NNNC"
+		(property "MPN" "CC0603KRX7R9BB104"
 			(at 0 0 270)
 			(unlocked yes)
@@
 			)
 		)
-		(property "LCSC PN" "C1590"
+		(property "LCSC PN" "C14663"
 			(at 0 0 0)
 			(unlocked yes)
@@
 			)
 		)
-		(property "Manufacturer" "Samsung Electro-Mechanics"
+		(property "Manufacturer" "Yageo"
 			(at 0 0 0)
 			(unlocked yes)
@@
 			)
 		)
-		(property "Manufacturer Part" "CL10B104KA8NNNC"
+		(property "Manufacturer Part" "CC0603KRX7R9BB104"
 			(at 0 0 0)
 			(unlocked yes)
@@
 			)
 		)
-		(property "MPN" "CL10B104KA8NNNC"
+		(property "MPN" "CC0603KRX7R9BB104"
 			(at 0 0 0)
 			(unlocked yes)
@@
 			)
 		)
-		(property "LCSC PN" "C1590"
+		(property "LCSC PN" "C14663"
 			(at 0 0 90)
 			(unlocked yes)
@@
 			)
 		)
-		(property "Manufacturer" "Samsung Electro-Mechanics"
+		(property "Manufacturer" "Yageo"
 			(at 0 0 90)
 			(unlocked yes)
@@
 			)
 		)
-		(property "Manufacturer Part" "CL10B104KA8NNNC"
+		(property "Manufacturer Part" "CC0603KRX7R9BB104"
 			(at 0 0 90)
 			(unlocked yes)
@@
 			)
 		)
-		(property "MPN" "CL10B104KA8NNNC"
+		(property "MPN" "CC0603KRX7R9BB104"
 			(at 0 0 90)
 			(unlocked yes)
@@
 			)
 		)
-		(property "LCSC PN" "C1590"
+		(property "LCSC PN" "C14663"
 			(at 0 0 270)
 			(unlocked yes)
@@
 			)
 		)
-		(property "Manufacturer" "Samsung Electro-Mechanics"
+		(property "Manufacturer" "Yageo"
 			(at 0 0 270)
 			(unlocked yes)
@@
 			)
 		)
-		(property "Manufacturer Part" "CL10B104KA8NNNC"
+		(property "Manufacturer Part" "CC0603KRX7R9BB104"
 			(at 0 0 270)
 			(unlocked yes)
@@
 			)
 		)
-		(property "MPN" "CL10B104KA8NNNC"
+		(property "MPN" "CC0603KRX7R9BB104"
 			(at 0 0 270)
 			(unlocked yes)
@@
 			)
 		)
-		(property "LCSC PN" "C1590"
+		(property "LCSC PN" "C14663"
 			(at 0 0 0)
 			(unlocked yes)
@@
 			)
 		)
-		(property "Manufacturer" "Samsung Electro-Mechanics"
+		(property "Manufacturer" "Yageo"
 			(at 0 0 0)
 			(unlocked yes)
@@
 			)
 		)
-		(property "MPN" "CL10B104KA8NNNC"
+		(property "MPN" "CC0603KRX7R9BB104"
 			(at 0 0 0)
 			(unlocked yes)
@@
 			)
 		)
+		(property "Manufacturer Part" "CC0603KRX7R9BB104"
+			(at 0 0 0)
+			(layer "F.Fab")
+			(hide yes)
+			(effects
+				(font
+					(size 1 1)
+					(thickness 0.15)
+				)
+			)
+		)
 		(property ki_fp_filters "C_*")
 		(sheetname "/SENSORES/")
@@
 			)
 		)
-		(property "LCSC PN" "C1590"
+		(property "LCSC PN" "C14663"
 			(at 0 0 270)
 			(unlocked yes)
@@
 			)
 		)
-		(property "Manufacturer" "Samsung Electro-Mechanics"
+		(property "Manufacturer" "Yageo"
 			(at 0 0 270)
 			(unlocked yes)
@@
 			)
 		)
-		(property "MPN" "CL10B104KA8NNNC"
+		(property "MPN" "CC0603KRX7R9BB104"
 			(at 0 0 270)
 			(unlocked yes)
@@
 			)
 		)
+		(property "Manufacturer Part" "CC0603KRX7R9BB104"
+			(at 0 0 0)
+			(layer "F.Fab")
+			(hide yes)
+			(effects
+				(font
+					(size 1 1)
+					(thickness 0.15)
+				)
+			)
+		)
 		(property ki_fp_filters "C_*")
 		(sheetname "/SENSORES/")
@@
 			)
 		)
-		(property "LCSC PN" "C1590"
+		(property "LCSC PN" "C14663"
 			(at 0 0 90)
 			(unlocked yes)
@@
 			)
 		)
-		(property "Manufacturer" "Samsung Electro-Mechanics"
+		(property "Manufacturer" "Yageo"
 			(at 0 0 90)
 			(unlocked yes)
@@
 			)
 		)
-		(property "MPN" "CL10B104KA8NNNC"
+		(property "MPN" "CC0603KRX7R9BB104"
 			(at 0 0 90)
 			(unlocked yes)
@@
 			)
 		)
+		(property "Manufacturer Part" "CC0603KRX7R9BB104"
+			(at 0 0 0)
+			(layer "F.Fab")
+			(hide yes)
+			(effects
+				(font
+					(size 1 1)
+					(thickness 0.15)
+				)
+			)
+		)
 		(property ki_fp_filters "C_*")
 		(sheetname "/SENSORES/")
@@
 			)
 		)
-		(property "Value" "1uF"
+		(property "Value" "100nF"
 			(at 0 1.43 0)
 			(layer "F.Fab")
@@
 			)
 		)
-		(property "LCSC PN" "C108463"
+		(property "LCSC PN" "C14663"
 			(at 0 0 180)
 			(unlocked yes)
@@
 			)
 		)
-		(property "Manufacturer" "Walsin Technology"
+		(property "Manufacturer" "Yageo"
 			(at 0 0 180)
 			(unlocked yes)
@@
 			)
 		)
-		(property "MPN" "0603B105K160CT"
+		(property "MPN" "CC0603KRX7R9BB104"
 			(at 0 0 180)
 			(unlocked yes)
@@
 			)
 		)
+		(property "Manufacturer Part" "CC0603KRX7R9BB104"
+			(at 0 0 0)
+			(layer "F.Fab")
+			(hide yes)
+			(effects
+				(font
+					(size 1 1)
+					(thickness 0.15)
+				)
+			)
+		)
 		(property ki_fp_filters "C_*")
 		(sheetname "/SENSORES/")
@@
 			)
 		)
-		(property "Value" "4.7k"
+		(property "Value" "47k"
 			(at 0 1.43 90)
 			(layer "F.Fab")
@@
 			)
 		)
-		(property "LCSC PN" "C23162"
+		(property "LCSC PN" "C25819"
 			(at 0 0 90)
 			(unlocked yes)
@@
 			)
 		)
-		(property "Manufacturer" "Walsin Technology"
+		(property "Manufacturer" "UNI-ROYAL"
 			(at 0 0 90)
 			(unlocked yes)
@@
 			)
 		)
-		(property "MPN" "0603WAF4701T5E"
+		(property "MPN" "0603WAF4702T5E"
 			(at 0 0 90)
 			(unlocked yes)
@@
 			)
 		)
+		(property "Manufacturer Part" "0603WAF4702T5E"
+			(at 0 0 0)
+			(layer "F.Fab")
+			(hide yes)
+			(effects
+				(font
+					(size 1 1)
+					(thickness 0.15)
+				)
+			)
+		)
 		(property ki_fp_filters "R_*")
 		(sheetname "/SENSORES/")
@@
 			)
 		)
-		(property "LCSC PN" "C1590"
+		(property "LCSC PN" "C14663"
 			(at 0 0 270)
 			(unlocked yes)
@@
 			)
 		)
-		(property "Manufacturer" "Samsung Electro-Mechanics"
+		(property "Manufacturer" "Yageo"
 			(at 0 0 270)
 			(unlocked yes)
@@
 			)
 		)
-		(property "Manufacturer Part" "CL10B104KA8NNNC"
+		(property "Manufacturer Part" "CC0603KRX7R9BB104"
 			(at 0 0 270)
 			(unlocked yes)
@@
 			)
 		)
-		(property "MPN" "CL10B104KA8NNNC"
+		(property "MPN" "CC0603KRX7R9BB104"
 			(at 0 0 270)
 			(unlocked yes)
@@
 			)
 		)
-		(property "LCSC PN" "C1590"
+		(property "LCSC PN" "C14663"
 			(at 0 0 270)
 			(unlocked yes)
@@
 			)
 		)
-		(property "Manufacturer" "Samsung Electro-Mechanics"
+		(property "Manufacturer" "Yageo"
 			(at 0 0 270)
 			(unlocked yes)
@@
 			)
 		)
-		(property "MPN" "CL10B104KA8NNNC"
+		(property "MPN" "CC0603KRX7R9BB104"
 			(at 0 0 270)
 			(unlocked yes)
@@
 			)
 		)
+		(property "Manufacturer Part" "CC0603KRX7R9BB104"
+			(at 0 0 0)
+			(layer "F.Fab")
+			(hide yes)
+			(effects
+				(font
+					(size 1 1)
+					(thickness 0.15)
+				)
+			)
+		)
 		(property ki_fp_filters "C_*")
 		(sheetname "/SENSORES/")
@@
 	)
 	(segment
+		(start 96.745 60.155)
+		(end 101.04 64.45)
+		(width 0.6)
+		(layer "F.Cu")
+		(net "/ALIMENTACION/3.3V_EXT")
+	)
+	(segment
+		(start 101.04 64.45)
+		(end 103.7 64.45)
+		(width 0.6)
+		(layer "F.Cu")
+		(net "/ALIMENTACION/3.3V_EXT")
+	)
+	(segment
 		(start 104.6 101.75)
 		(end 110.053408 101.75)
@@
 		(net "Net-(U7B--)")
 	)
-	(segment
-		(start 96.745 60.155)
-		(end 101.04 64.45)
-		(width 0.6)
-		(layer "F.Cu")
-		(net "/ALIMENTACION/3.3V_EXT")
-	)
-	(segment
-		(start 101.04 64.45)
-		(end 103.7 64.45)
-		(width 0.6)
-		(layer "F.Cu")
-		(net "/ALIMENTACION/3.3V_EXT")
-	)
 	(zone
