File: PCB_SALUS_v3.kicad_pcb (KiCad board)
At the start: 2 copper layers, 100 x 100 mm, 87 parts, among them J1 Debug_U0, J10 RELES_2, J11 Throttle, J12 I2C_EXT1, J13 I2C_EXT2, J14 S_HALL, J15 RF_PPM, J16 USB_NATIVO, J17 SERVO2, J18 SERVO1, J19 +7V_IN, J2 S_GIRO, J20 3V_IN, J21 RS485, J22 GPIOS_AUX, J3 RS485, J4 Uart1, J5 5V_IN, J6 IBT_2, J7 FC1, J8 FC2, J9 RELES_1, U1 AMS1117CD-3.3, U2 SP3485EN, U4 BMI088, U5 74HC595, U6 ULN2003A, U7 LM358, U8 ESP32-S3-WROOM-1

Commit message: Registra PCB SALUS v3 con montaje M3 y terminacion RS485
Conserva los dos paquetes de fabricacion del 20 de agosto, sus fuentes, checksums y validaciones. El paquete final monta R4 de 120 ohm e incluye 64 componentes SMD. Actualiza el README para identificar la entrega vigente y los limites de la validacion archivada.
Parts:
- added H1: MountingHole_3.2mm_M3, MountingHole:MountingHole_3.2mm_M3, F.Cu at (145.0, 145.0)
- added H2: MountingHole_3.2mm_M3, MountingHole:MountingHole_3.2mm_M3, F.Cu at (145.5, 55.0)
- added H3: MountingHole_3.2mm_M3, MountingHole:MountingHole_3.2mm_M3, F.Cu at (55.0, 55.0)
- added H4: MountingHole_3.2mm_M3, MountingHole:MountingHole_3.2mm_M3, F.Cu at (55.0, 145.0)
