File: ALIMENTACION.kicad_sch (KiCad schematic)
At the start: 11 parts, among them J20 3V_IN, J5 5V_IN, U1 AMS1117CD-3.3

Commit message: Deshabilita alimentacion USB con D9 DNP y actualiza entrega
Parts:
- D9: BOM Comments (none) -> D9 NO MONTAR: alimentacion USB deshabilitada. No sustituir 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; now not fitted; now left out of the parts list
Changed lines of the file:
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@@
 		(body_style 1)
 		(exclude_from_sim no)
-		(in_bom yes)
+		(in_bom no)
 		(on_board yes)
-		(in_pos_files yes)
-		(dnp no)
+		(in_pos_files no)
+		(dnp yes)
 		(fields_autoplaced yes)
+		(property "BOM Comments" "D9 NO MONTAR: alimentacion USB deshabilitada. No sustituir por puente." (at 53.34 111.76 0) (effects (font (size 1.27 1.27)) (hide yes)))
 		(property "Reference" "D9"
 			(at 53.6575 105.41 0)
