File: _restore_backup_2026-08-03T13-33-40-644/ESP32.kicad_sch (KiCad schematic)
At the start: 25 parts, among them J1 Debug_U0, J16 USB_NATIVO, J3 RS485, J4 Uart1, U2 SP3485EN, U8 ESP32-S3-WROOM-1

Commit message: RS485
Parts:
- removed C7: 100nF, Capacitor_SMD:C_0603_1608Metric, symbol Device:C
- removed J3: RS485, Connector_PinHeader_2.54mm:PinHeader_1x04_P2.54mm_Vertical, symbol Connector_Generic:Conn_01x04
- removed R37: 10k, Resistor_SMD:R_0603_1608Metric, symbol Device:R
- removed U2: SP3485EN, Package_SO:SOIC-8_3.9x4.9mm_P1.27mm, symbol Interface_UART:SP3485EN
Connections:
- net RS485_DIR: no longer names the net of U8.35 (IO42)
- no-connect marks 7 -> 8
Other:
- note removed: "RS485"
